Commit message: Fix URDF dimensions from photos, add Gazebo stabilizers, update configs
Corrected robot dimensions using 8x8" base plate as reference:
- wheel_separation: 0.50 -> 0.30m (estimated from motor mount offsets)
- chassis: 0.35x0.30x0.20 -> 0.203x0.203x0.28m (3 plates, 10-12" tall)
- chassis_z_offset: 0.02 -> 0.14m (centered in taller chassis)
- camera_z: 1.27 -> 1.63m (recalculated from new chassis height + mast)
- imu_z: 0.12 -> 0.22m (near top plate of 3-plate stack)
- robot_radius: 0.30 -> 0.22m in Nav2 costmaps
- Added mast_y_offset for side-mounted mast bracket (per photos)

Added invisible frictionless stabilizer spheres for Gazebo sim (use_sim
only) to prevent the two-wheeled robot from tipping. Changed use_sim
from fixed property to xacro arg so gazebo.launch.py can enable it.

Updated EKF comments documenting BNO085 rotation vector mode usage.
All estimated values marked [TENTATIVE] for hardware verification.

https://claude.ai/code/session_01G5mLqXmgaVQSMU8RGYon1Q

File: johnny5_description/urdf/chassis.urdf.xacro (robot description, xacro)
@@ -33,11 +33,11 @@
     </link>
   </xacro:macro>
-  <!-- Mast macro: carbon fiber survey pole -->
+  <!-- Mast macro: carbon fiber survey pole (LS2015) -->
   <xacro:macro name="mast">
     <joint name="chassis_to_mast" type="fixed">
       <parent link="chassis_link"/>
       <child link="mast_link"/>
-      <!-- mast base at top of chassis, slightly behind center -->
-      <origin xyz="-0.05 0 ${chassis_height/2 + mast_height/2}" rpy="0 0 0"/>
+      <!-- [TENTATIVE] mast base at top of chassis; x/y offset estimated from photos -->
+      <origin xyz="${mast_x_offset} ${mast_y_offset} ${chassis_height/2 + mast_height/2}" rpy="0 0 0"/>
     </joint>
     <link name="mast_link">

File: johnny5_description/urdf/gazebo.urdf.xacro (robot description, xacro)
@@ -32,4 +32,51 @@
     <material>Gazebo/Grey</material>
   </gazebo>
+  <!-- ==================== Sim-Only Stabilizers ==================== -->
+  <!-- Invisible frictionless spheres at front/rear prevent the       -->
+  <!-- two-wheeled robot from tipping in Gazebo. ~5mm ground gap     -->
+  <!-- allows ~3.5 deg tilt before contact. No visual = invisible    -->
+  <!-- in RViz. On real hardware, the Teensy balance controller       -->
+  <!-- handles stability; these only exist when use_sim:=true.        -->
+  <xacro:if value="${use_sim}">
+    <link name="front_stabilizer_link">
+      <collision>
+        <geometry><sphere radius="0.005"/></geometry>
+      </collision>
+      <inertial>
+        <mass value="0.001"/>
+        <inertia ixx="1e-8" ixy="0" ixz="0" iyy="1e-8" iyz="0" izz="1e-8"/>
+      </inertial>
+    </link>
+    <joint name="front_stabilizer_joint" type="fixed">
+      <parent link="base_link"/>
+      <child link="front_stabilizer_link"/>
+      <!-- z = -(wheel_radius - sphere_radius - 5mm gap) -->
+      <origin xyz="0.09 0 -0.0726" rpy="0 0 0"/>
+    </joint>
+    <gazebo reference="front_stabilizer_link">
+      <mu1>0.0</mu1>
+      <mu2>0.0</mu2>
+      <material>Gazebo/White</material>
+    </gazebo>
+    <link name="rear_stabilizer_link">
+      <collision>
+        <geometry><sphere radius="0.005"/></geometry>
+      </collision>
+      <inertial>
+        <mass value="0.001"/>
+        <inertia ixx="1e-8" ixy="0" ixz="0" iyy="1e-8" iyz="0" izz="1e-8"/>
+      </inertial>
+    </link>
+    <joint name="rear_stabilizer_joint" type="fixed">
+      <parent link="base_link"/>
+      <child link="rear_stabilizer_link"/>
+      <origin xyz="-0.09 0 -0.0726" rpy="0 0 0"/>
+    </joint>
+    <gazebo reference="rear_stabilizer_link">
+      <mu1>0.0</mu1>
+      <mu2>0.0</mu2>
+      <material>Gazebo/White</material>
+    </gazebo>
+  </xacro:if>
   <!-- ==================== Differential Drive ==================== -->
   <!-- Approximates the two-wheeled balance bot for Nav2 testing.   -->

File: johnny5_description/urdf/johnny5.urdf.xacro (robot description, xacro)
@@ -9,23 +9,39 @@
   <!--   base_link = center of wheel axle                          -->
   <!-- ============================================================ -->
-  <!-- Global properties -->
-  <xacro:property name="wheel_radius"     value="0.08255"/>  <!-- 6.5" / 2 -->
-  <xacro:property name="wheel_width"      value="0.055"/>
-  <xacro:property name="wheel_mass"       value="1.8"/>      <!-- hoverboard hub motor -->
-  <xacro:property name="wheel_separation" value="0.50"/>     <!-- track width center-to-center -->
-  <xacro:property name="chassis_length"   value="0.35"/>     <!-- x -->
-  <xacro:property name="chassis_width"    value="0.30"/>     <!-- y -->
-  <xacro:property name="chassis_height"   value="0.20"/>     <!-- z total deck stack -->
-  <xacro:property name="chassis_mass"     value="8.0"/>      <!-- batteries+ESC+Jetson+structure -->
-  <xacro:property name="chassis_z_offset" value="0.02"/>     <!-- center of mass above axle -->
-  <xacro:property name="mast_radius"      value="0.016"/>    <!-- 32mm diameter -->
-  <xacro:property name="mast_height"      value="1.35"/>     <!-- 3 x 0.45m sections -->
-  <xacro:property name="mast_mass"        value="0.5"/>
-  <xacro:property name="lidar_x"          value="0.10"/>     <!-- forward of base_link -->
-  <xacro:property name="lidar_z"          value="0.10"/>     <!-- ~18cm above ground -->
-  <xacro:property name="imu_x"            value="0.0"/>
-  <xacro:property name="imu_z"            value="0.12"/>     <!-- upper deck -->
-  <xacro:property name="camera_z"         value="1.27"/>     <!-- mast top above axle -->
-  <xacro:property name="use_sim" value="false"/>
+  <!-- ============================================================ -->
+  <!-- TENTATIVE DIMENSIONS - Estimated from photos + 8x8" base    -->
+  <!-- plates. All values marked [TENTATIVE] need physical          -->
+  <!-- measurement on hardware to verify.                           -->
+  <!-- ============================================================ -->
+  <!-- Simulation mode (set via xacro arg: use_sim:=true) -->
+  <xacro:arg name="use_sim" default="false"/>
+  <xacro:property name="use_sim" value="$(arg use_sim)"/>
+  <!-- Wheels: 6.5" Gyroor hoverboard hub motors (BOM-confirmed) -->
+  <xacro:property name="wheel_radius"     value="0.08255"/>  <!-- 6.5" / 2 — confirmed from BOM -->
+  <xacro:property name="wheel_width"      value="0.055"/>    <!-- [TENTATIVE] ~2.2", needs measurement -->
+  <xacro:property name="wheel_mass"       value="1.8"/>      <!-- [TENTATIVE] hoverboard hub motor w/ magnets+windings -->
+  <xacro:property name="wheel_separation" value="0.30"/>     <!-- [TENTATIVE] ~12" — 8" plate + 2x motor mount offset -->
+  <!-- Chassis: 3x 8x8" aluminum plates with standoffs -->
+  <xacro:property name="chassis_length"   value="0.203"/>    <!-- 8" = 203mm — confirmed by user -->
+  <xacro:property name="chassis_width"    value="0.203"/>    <!-- 8" = 203mm — confirmed by user -->
+  <xacro:property name="chassis_height"   value="0.28"/>     <!-- [TENTATIVE] ~11" — 3 plates + standoffs, user says 10-12" -->
+  <xacro:property name="chassis_mass"     value="8.0"/>      <!-- [TENTATIVE] batteries+ESC+Jetson+3 plates+standoffs -->
+  <xacro:property name="chassis_z_offset" value="0.14"/>     <!-- [TENTATIVE] chassis_height/2, assumes bottom plate at axle -->
+  <!-- Mast: LS2015 carbon fiber survey pole, 4-section, 1.8m total -->
+  <xacro:property name="mast_radius"      value="0.016"/>    <!-- 32mm diameter — from BOM (LS2015) -->
+  <xacro:property name="mast_height"      value="1.35"/>     <!-- 3 x 0.45m sections (standard config) -->
+  <xacro:property name="mast_mass"        value="0.5"/>      <!-- [TENTATIVE] carbon fiber pole + connectors -->
+  <xacro:property name="mast_x_offset"    value="-0.05"/>    <!-- [TENTATIVE] slightly behind center -->
+  <xacro:property name="mast_y_offset"    value="0.07"/>     <!-- [TENTATIVE] offset to one side per photos -->
+  <!-- LiDAR: LDROBOT STL-19P — not yet mounted, position TBD -->
+  <xacro:property name="lidar_x"          value="0.10"/>     <!-- [TENTATIVE] forward of base_link -->
+  <xacro:property name="lidar_z"          value="0.10"/>     <!-- [TENTATIVE] design spec: 6-8" above ground -->
+  <!-- IMU: BNO085 on Teensy breakout, upper deck area -->
+  <xacro:property name="imu_x"            value="0.0"/>      <!-- [TENTATIVE] assumed centered -->
+  <xacro:property name="imu_z"            value="0.22"/>     <!-- [TENTATIVE] near top plate of 3-plate stack -->
+  <!-- Camera: OAK-D Pro at mast top -->
+  <!-- camera_z = chassis_z_offset + chassis_height/2 + mast_height -->
+  <!--         = 0.14 + 0.14 + 1.35 = 1.63m above base_link        -->
+  <xacro:property name="camera_z"         value="1.63"/>     <!-- [TENTATIVE] depends on mast config + chassis height -->
   <!-- Include sub-files -->
   <xacro:include filename="$(find johnny5_description)/urdf/chassis.urdf.xacro"/>
